File: hardware/sim_card_tester/schematic.sch (EAGLE design)
At the start: 139 parts, among them IC1 TPS6300, J1 CON_MICRO_SDDM3AT-SF-PEJM5, J2 MICRO_USB_B_HIROSE_ZX62R-B-5P, J3 NANO_SIM, J4 NANO_SIM, J5 NANO_SIM, J6 NANO_SIM, J7 TC2030-JLINK-L, J8 U.FL-R-SMT, Q1 MOSFET-NCHANNELSMD, Q2 MOSFET-NCHANNELSMD, Q3 MOSFET-NCHANNELSMD, Q4 SI223DDS, U1 AB1815-T3, U10 SIP32510, U11 SIP32510, U12 UBLOX_SARA_G350, U13 TXB0104RUT, U15 MAX4734EUB+, U2 BGA725L6-ALT, U20 MAX4734EUB+, U21 MAX4734EUB+, U22 MAX4734EUB+, U3 FTDI234XD, U4 SAFFB1G56KB0F0A, U5 MAX8887EZK33+T, U6 MCP73831, U7 MAX-M8, U8 MAX67XXMAX6749MAX67XX, U9 NRF52840, X1 ABS07-32.768KHZ-7-T, X4 32MHz, X5 32.768kHz

Commit message: renumbering again
Parts:
- C22: DIGIKEY 490-5405-1-ND -> 490-6328-1-ND; MPN GRM033R61A104ME15D -> GRM155R71C104KA88J
- C23, C27: DIGIKEY (none) -> 490-6328-1-ND; MANUFACTURER (none) -> Murata Electronics; MPN (none) -> GRM155R71C104KA88J
- C24, C25, C26: MANUFACTURER (none) -> Murata Electronics
- C32: DIGIKEY (none) -> 399-3118-1-ND; MANUFACTURER (none) -> KEMET; MPN (none) -> C0603C105K8PACTU
- C33: DIGIKEY 490-7195-1-ND -> 399-3118-1-ND; MANUFACTURER (none) -> KEMET; MPN GRM155R70G105KA12D -> C0603C105K8PACTU
- renumbered U$5 to C50
Changed lines of the file:
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@@
 </part>
 <part name="C22" library="Nordic_nRF" library_urn="urn:adsk.eagle:library:169009" deviceset="CAPACITOR" device="_0603_L" package3d_urn="urn:adsk.eagle:package:2593727/1" value="0.1uF">
-<attribute name="DIGIKEY" value="490-5405-1-ND"/>
+<attribute name="DIGIKEY" value="490-6328-1-ND"/>
 <attribute name="MANUFACTURER" value="Murata Electronics"/>
-<attribute name="MPN" value="GRM033R61A104ME15D"/>
+<attribute name="MPN" value="GRM155R71C104KA88J "/>
 </part>
 <part name="C41" library="Nordic_nRF" library_urn="urn:adsk.eagle:library:169009" deviceset="CAPACITOR" device="_0603_L" package3d_urn="urn:adsk.eagle:package:2593727/1" value="10uF">
@@
 <attribute name="MPN" value="RC0603JR-072M2L"/>
 </part>
-<part name="C23" library="Nordic_nRF" library_urn="urn:adsk.eagle:library:169009" deviceset="CAPACITOR" device="_0603_L" package3d_urn="urn:adsk.eagle:package:2593727/1" value="0.1uF"/>
+<part name="C23" library="Nordic_nRF" library_urn="urn:adsk.eagle:library:169009" deviceset="CAPACITOR" device="_0603_L" package3d_urn="urn:adsk.eagle:package:2593727/1" value="0.1uF">
+<attribute name="DIGIKEY" value="490-6328-1-ND"/>
+<attribute name="MANUFACTURER" value="Murata Electronics"/>
+<attribute name="MPN" value="GRM155R71C104KA88J "/>
+</part>
 <part name="SUPPLY2" library="supply1" library_urn="urn:adsk.eagle:library:371" deviceset="GND" device=""/>
 <part name="SUPPLY3" library="supply1" library_urn="urn:adsk.eagle:library:371" deviceset="GND" device=""/>
@@
 <attribute name="MPN" value="RC0603FR-07100RL"/>
 </part>
-<part name="U$5" library="Nordic_nRF" library_urn="urn:adsk.eagle:library:169009" deviceset="CAPACITOR" device="_0603_L" package3d_urn="urn:adsk.eagle:package:2593727/1" value=".1uF"/>
+<part name="C50" library="Nordic_nRF" library_urn="urn:adsk.eagle:library:169009" deviceset="CAPACITOR" device="_0603_L" package3d_urn="urn:adsk.eagle:package:2593727/1" value=".1uF"/>
 <part name="GND8" library="SparkFun-PowerSymbols" deviceset="GND" device=""/>
 <part name="R36" library="BeagleBone_Black_Wireless" library_urn="urn:adsk.eagle:library:6644236" deviceset="R-US_" device="R0603" package3d_urn="urn:adsk.eagle:package:8118505/1" value="1.3M">
@@
 <part name="U9" library="chips" deviceset="NRF52840" device=""/>
 <part name="C32" library="Nordic_nRF" library_urn="urn:adsk.eagle:library:169009" deviceset="CAPACITOR" device="_0603_L" package3d_urn="urn:adsk.eagle:package:2593727/1" value="1uF">
-<attribute name="DIGIKEY" value=""/>
-<attribute name="MPN" value=""/>
+<attribute name="DIGIKEY" value="399-3118-1-ND"/>
+<attribute name="MANUFACTURER" value="KEMET"/>
+<attribute name="MPN" value="C0603C105K8PACTU"/>
 </part>
 <part name="C24" library="Nordic_nRF" library_urn="urn:adsk.eagle:library:169009" deviceset="CAPACITOR" device="_0603_L" package3d_urn="urn:adsk.eagle:package:2593727/1" value="0.1uF">
 <attribute name="DIGIKEY" value="490-6328-1-ND"/>
+<attribute name="MANUFACTURER" value="Murata Electronics"/>
 <attribute name="MPN" value="GRM155R71C104KA88J "/>
 </part>
@@
 <part name="C25" library="Nordic_nRF" library_urn="urn:adsk.eagle:library:169009" deviceset="CAPACITOR" device="_0603_L" package3d_urn="urn:adsk.eagle:package:2593727/1" value="0.1uF">
 <attribute name="DIGIKEY" value="490-6328-1-ND"/>
+<attribute name="MANUFACTURER" value="Murata Electronics"/>
 <attribute name="MPN" value="GRM155R71C104KA88J "/>
 </part>
 <part name="C26" library="Nordic_nRF" library_urn="urn:adsk.eagle:library:169009" deviceset="CAPACITOR" device="_0603_L" package3d_urn="urn:adsk.eagle:package:2593727/1" value="0.1uF">
 <attribute name="DIGIKEY" value="490-6328-1-ND"/>
+<attribute name="MANUFACTURER" value="Murata Electronics"/>
 <attribute name="MPN" value="GRM155R71C104KA88J "/>
 </part>
 <part name="C27" library="Nordic_nRF" library_urn="urn:adsk.eagle:library:169009" deviceset="CAPACITOR" device="_0603_L" package3d_urn="urn:adsk.eagle:package:2593727/1" value="0.1uF">
-<attribute name="DIGIKEY" value=""/>
-<attribute name="MPN" value=""/>
+<attribute name="DIGIKEY" value="490-6328-1-ND"/>
+<attribute name="MANUFACTURER" value="Murata Electronics"/>
+<attribute name="MPN" value="GRM155R71C104KA88J "/>
 </part>
 <part name="C14" library="Nordic_nRF" library_urn="urn:adsk.eagle:library:169009" deviceset="CAPACITOR" device="_0603_L" package3d_urn="urn:adsk.eagle:package:2593727/1" value="100pF">
@@
 <part name="X4" library="crystals" deviceset="7V" device="-32.000MAHV-T" value="32MHz"/>
 <part name="C33" library="Nordic_nRF" library_urn="urn:adsk.eagle:library:169009" deviceset="CAPACITOR" device="_0603_L" package3d_urn="urn:adsk.eagle:package:2593727/1" value="1uF">
-<attribute name="DIGIKEY" value="490-7195-1-ND "/>
-<attribute name="MPN" value="GRM155R70G105KA12D "/>
+<attribute name="DIGIKEY" value="399-3118-1-ND"/>
+<attribute name="MANUFACTURER" value="KEMET"/>
+<attribute name="MPN" value="C0603C105K8PACTU"/>
 </part>
 <part name="GND20" library="supply1" library_urn="urn:adsk.eagle:library:371" deviceset="GND" device=""/>
@@
 <attribute name="NAME" x="598.17" y="110.49" size="1.778" layer="95" ratio="12" rot="R90" align="bottom-center"/>
 <attribute name="VALUE" x="600.71" y="110.49" size="1.778" layer="96" ratio="12" rot="R270" align="bottom-center"/>
+<attribute name="MANUFACTURER" x="599.44" y="111.76" size="1.778" layer="96"/>
 </instance>
 <instance part="C26" gate="C$1" x="739.14" y="144.78" smashed="yes">
@@
 <attribute name="NAME" x="31.496" y="-17.78" size="1.778" layer="95" font="vector" rot="R90" align="bottom-center"/>
 </instance>
-<instance part="U$5" gate="C$1" x="33.02" y="-27.94" smashed="yes">
+<instance part="C50" gate="C$1" x="33.02" y="-27.94" smashed="yes">
 <attribute name="NAME" x="34.544" y="-27.559" size="1.778" layer="95"/>
 <attribute name="VALUE" x="34.544" y="-32.639" size="1.778" layer="96"/>
@@
 </segment>
 <segment>
-<pinref part="U$5" gate="C$1" pin="2"/>
+<pinref part="C50" gate="C$1" pin="2"/>
 <pinref part="GND8" gate="1" pin="GND"/>
 </segment>
@@
 <segment>
 <pinref part="R5" gate="G$1" pin="1"/>
-<pinref part="U$5" gate="C$1" pin="1"/>
+<pinref part="C50" gate="C$1" pin="1"/>
 <wire x1="33.02" y1="-22.86" x2="33.02" y2="-25.4" width="0.1524" layer="91"/>
 <wire x1="33.02" y1="-25.4" x2="43.18" y2="-25.4" width="0.1524" layer="91"/>

Commit message: fixed numbering
Parts:
- removed C50: .1uF, Nordic_nRF:CAPACITOR_0603_L
- added C47: 220uF, BeagleBone_Black_Wireless:C-USC1210
- C28: value 100nF -> .1uF; DIGIKEY 490-5405-1-ND -> (none); MANUFACTURER Murata Electronics -> (none); MPN GRM033R61A104ME15D -> (none)
- C29: DESCRIPTION CAP CER 0.1UF 10V X7R 0402 -> (none); DIGIKEY 490-10777-1-ND -> 490-5405-1-ND; MANUFACTURER Murata -> Murata Electronics; MPN GRM155R71A104JA01D -> GRM033R61A104ME15D
- C30: value 0.82uF -> 100nF; DESCRIPTION (none) -> CAP CER 0.1UF 10V X7R 0402; DIGIKEY 399-3117-1-ND -> 490-10777-1-ND; MANUFACTURER KEMET -> Murata; MPN C0603C824K8PACTU -> GRM155R71A104JA01D
- C31: value 1uF -> 0.82uF; device passives:CAPACITOR0402_CAP -> Nordic_nRF:CAPACITOR_0603_L; DIGIKEY 399-3118-1-ND -> 399-3117-1-ND; MPN C0603C105K8PACTU -> C0603C824K8PACTU
- C32: device Nordic_nRF:CAPACITOR_0603_L -> passives:CAPACITOR0402_CAP
- C34: value 2.2uF -> 1uF; DIGIKEY 490-12738-1-ND -> 399-3118-1-ND; MANUFACTURER Murata Electronics -> KEMET; MPN GRM188R61E225MA12D -> C0603C105K8PACTU
- C35: value 4.7uF -> 2.2uF; DIGIKEY 490-10992-1-ND -> 490-12738-1-ND; MPN ZRB18AR6YA475KE05L -> GRM188R61E225MA12D
- C41: value 10uF -> 4.7uF; DIGIKEY 490-14372-1-ND -> 490-10992-1-ND; MPN GRM188R60J106KE47D -> ZRB18AR6YA475KE05L
- C42: DIGIKEY 490-12538-1-ND -> 490-14372-1-ND
- C45: value 100uF -> 10uF; device BeagleBone_Black_Wireless:C-USC1210 -> Nordic_nRF:CAPACITOR_0603_L; DIGIKEY 490-9969-1-ND -> 490-12538-1-ND; MPN GRM32ER61A107ME20L -> GRM188R60J106KE47D
- C46: value 220uF -> 100uF; DIGIKEY 490-16308-1-ND -> 490-9969-1-ND; MPN GRM32ER60J227ME05L -> GRM32ER61A107ME20L
Connections:
- net +3V3: now also C33.1, C36.1, C40.1, C45.1; no longer C31.1, C35.1, C37.1, C43.1
- net BAT: now also C37.1, C43.1; no longer C36.1, C42.1
- net GND: now also C41.2, C42.1, C47.2; no longer C41.1, C42.2, C50.2
- net GPS_VCC: now also C42.2; no longer C41.2
- net GSM_GATED: now also C30.1, C47.1; no longer C29.1, C46.1
- net N$16: now also C46.1; no longer C45.1
- net N$29: now also C28.1; no longer C50.1
- net N$32: now also C34.1; no longer C33.1
- net N$36: now also C31.1; no longer C30.1
- net N$39: now also C35.1; no longer C34.1
- net N$55: now also C41.1; no longer C40.1
- net VCC_LINUX_1V8: now also C29.1; no longer C28.1
Other:
- moved on the sheet: C33, C36, C37, C38, C43, C44, C46

Commit message: cleaned up wires
Connections:
- removed net +3V3: C24.1, C26.1, C27.1, C32.1, C33.1, C36.1, C38.1, C39.1, C40.1, C44.1, C45.1, D2.VDD, IC1G$1.VOUT, J7.VCC, Q4.S, R11.2, R14.1, R15.1, R25.2, R35.1, R36.2, TP15.TP, U1.VCC, U10.VSUPP, U11.VSUPP, U13.VCC_B, U5.!SHDN, U5.IN, U5.OUT, U6.VDD/1, U6.VDD/2, U9.VDD, U9.VDDH
- removed net VCC_LINUX_1V8: C29.1, U3.VCCIO
- new net 5V: C36.1, FB1.P$2, J2.+5V, R11.2, R35.1, U15.V+, U20.V+, U21.V+, U22.V+, U6.VDD/1, U6.VDD/2
- new net VCCA: C38.1, C44.1, C45.1, IC1G$1.VOUT, Q4.S, R36.2, U5.!SHDN, U5.IN
- net VCC: now also C24.1, C26.1, C27.1, C29.1, C32.1, C33.1, C39.1, C40.1, D2.VDD, J7.VCC, R14.1, R15.1, R25.2, TP15.TP, U1.VCC, U10.VSUPP, U11.VSUPP, U13.VCC_B, U3.VCCIO, U5.OUT, U9.VDD, U9.VDDH; no longer FB1.P$2, J2.+5V, U15.V+, U20.V+, U21.V+, U22.V+
Other:
- note added: "VCCA = 3.8V"

Commit message: added test points
Parts:
- added TP1, TP10, TP11, TP12, TP16, TP17, TP18, TP19, TP2, TP20, TP21, TP22, TP23, TP24, TP25, TP26, TP27, TP28, TP29, TP3, TP30, TP4, TP5, TP6, TP7, TP8, TP9: TEST-POINT, headers:TEST-POINT
- added TP31: TPTP06SQ, testpad:TPTP06SQ
- TP15: value TPTP06SQ -> TEST-POINT; device testpad:TPTP06SQ -> headers:TEST-POINT
Connections:
- net !EXTERNAL_RST: now also TP12.TESTPOINT
- net !NRF_CS_SD: now also TP11.TESTPOINT
- net !NRF_RST: now also TP13.TESTPOINT
- net !RTC_CS: now also TP4.TESTPOINT
- net !RTC_INT1: now also TP8.TESTPOINT
- net !SD_DETECT: now also TP21.TESTPOINT
- net BATIN: now also TP22.TESTPOINT
- net GND: now also TP28.TESTPOINT
- net GPS_PWR_EN: now also TP10.TESTPOINT
- net GPS_RXD: now also TP1.TESTPOINT
- net GPS_TXD: now also TP2.TESTPOINT
- net GSM_CTS: now also TP16.TESTPOINT
- net GSM_POWER: now also TP17.TESTPOINT
- net GSM_RST: now also TP19.TESTPOINT
- net GSM_RTS: now also TP18.TESTPOINT
- net GSM_TX: now also TP20.TESTPOINT
- net MUX_EN: now also TP9.TESTPOINT
- net MUX_SEL1: now also TP23.TESTPOINT
- net MUX_SEL2: now also TP26.TESTPOINT
- net NRF_GPIO_0: now also TP29.TESTPOINT; no longer TP13.TESTPOINT
- net NRF_GPIO_1: now also TP30.TESTPOINT; no longer TP14.TESTPOINT
- net NRF_MISO: now also TP7.TESTPOINT
- net NRF_MOSI: now also TP5.TESTPOINT
- net NRF_SWDCLK: now also TP15.TESTPOINT
- net NRF_SWDIO: now also TP14.TESTPOINT
- net SD_EN: now also TP6.TESTPOINT
- net UART_RX: now also TP24.TESTPOINT
- net UART_TX: now also TP25.TESTPOINT
- net VCC: now also TP27.TESTPOINT, TP31.TP; no longer TP15.TP
- net WDI: now also TP3.TESTPOINT

Commit message: updated bom
Parts:
- C22, C23, C24, C25, C26, C27: DIGIKEY 490-6328-1-ND -> 490-5405-1-ND; MPN GRM155R71C104KA88J -> GRM033R61A104ME15D
- C28: DIGIKEY (none) -> 490-5405-1-ND; MANUFACTURER (none) -> Murata Electronics; MPN (none) -> GRM033R61A104ME15D
- C29: value 100nF -> .1uF
- C30: value 100nF -> .1uF; DESCRIPTION CAP CER 0.1UF 10V X7R 0402 -> (none); DIGIKEY 490-10777-1-ND -> 490-5405-1-ND; MANUFACTURER Murata -> Murata Electronics; MPN GRM155R71A104JA01D -> GRM033R61A104ME15D
- C32: device passives:CAPACITOR0402_CAP -> Nordic_nRF:CAPACITOR_0603_L
- C42: DIGIKEY 490-14372-1-ND -> 490-12538-1-ND
- C6: device passives:CAPACITOR0402_CAP -> Nordic_nRF:CAPACITOR_0603_L; DIGIKEY 311-1065-1-ND -> 399-3118-1-ND; MANUFACTURER Yageo -> KEMET; MPN CC0603JRNPO9BN470 -> C0603C105K8PACTU
